Commit message: Update + Gazebo

File: phantomx_arm_description/urdf/phantomx.urdf (robot description, URDF)
Before this commit: robot phantomx_arm, 9 links, 8 joints
Joints:
- joint joint_1: origin xyz=0.396 0.526 0.35 rpy=1.570795 6.28318 1.570795 -> xyz=0.005 -0.13 0.35 rpy=1.570795 6.28318 3.14159
- joint joint_4: origin xyz=0.0 0.4268 0.0 rpy=3.14159 0.0 0.0 -> xyz=0.0 0.4268 0.0 rpy=6.28318 6.28318 0
- joint joint_5: limit (none) -> lower=-0.31 upper=0.1 effort=0 velocity=0.5; origin xyz=0.0 -0.28 0.0 rpy=1.570795 -1.570795 0.0 -> xyz=0.0 0.28 0.0 rpy=-1.570795 -1.570795 0.0

File: phantomx_arm_description/urdf/phantomx_macro.xacro (robot description, xacro)
@@ -4,5 +4,4 @@
    <property name="M_SCALE" value="0.04"/>
    <xacro:include filename="$(find phantomx_arm_description)/urdf/common_materials.xacro" />
-   <!-- Import all Gazebo-customization elements, including Gazebo colors -->
    <link name="world" />
    <joint name="fixed" type="fixed">
@@ -14,5 +13,5 @@
       <link name="${prefix}base_link">
          <visual>
-            <origin xyz="0 0 0" rpy="0 0 0" />
+            <origin xyz="${M_SCALE*10} ${M_SCALE*10} ${M_SCALE*0}" rpy="${M_PI*0} ${M_PI*0} ${M_PI}" />
             <geometry>
                <mesh filename="package://phantomx_arm_description/meshes/visual/base_link.stl" scale="${M_SCALE} ${M_SCALE} ${M_SCALE}"/>
@@ -20,5 +19,5 @@
 	    <xacro:material_black />
          </visual>
-         <collision> Setup Assistant will work for a few second before presenting you the results of its computation in the main table.
+         <collision>
             <origin xyz="0 0 0" rpy="0 0 0" />
             <geometry>
@@ -53,5 +52,5 @@
       </link>
       <link name="${prefix}link_2">
-         <visual>
+         <visual>with
             <origin xyz="0 0 0" rpy="0 0 0" />
             <geometry>
@@ -94,5 +93,5 @@
       <link name="${prefix}link_4">
          <visual>
-            <origin xyz="${M_SCALE*-1.18} ${M_SCALE*-3.3} ${M_SCALE*0}" rpy="0 0 0" />
+            <origin xyz="${M_SCALE*-1.18} ${M_SCALE*3.3} ${M_SCALE*0}" rpy="${M_PI*0} ${M_PI} ${-M_PI}" />
             <geometry>
                <mesh filename="package://phantomx_arm_description/meshes/visual/wrist_link.stl" scale="${M_SCALE} ${M_SCALE} ${M_SCALE}"/>
@@ -174,5 +173,5 @@
       <!-- joints -->
       <joint name="${prefix}joint_1" type="revolute">
-         <origin xyz="${M_SCALE*9.9} ${M_SCALE*13.15} ${M_SCALE*8.75}" rpy="${M_PI/2} ${M_PI*2} ${M_PI/2}" />
+         <origin xyz="${M_SCALE*0.125} ${M_SCALE*-3.25} ${M_SCALE*8.75}" rpy="${M_PI/2} ${M_PI*2} ${M_PI}" />
          <parent link="${prefix}base_link" />
          <child link="${prefix}link_1" />
@@ -195,5 +194,5 @@
       </joint>
       <joint name="${prefix}joint_4" type="revolute">
-         <origin xyz="${M_SCALE*0} ${M_SCALE*10.67} ${M_SCALE*0}" rpy="${M_PI} ${M_PI*0} ${M_PI*0}" />
+         <origin xyz="${M_SCALE*0} ${M_SCALE*10.67} ${M_SCALE*0}" rpy="${M_PI*2} ${M_PI*2} 0" />
          <parent link="${prefix}link_3" />
          <child link="${prefix}link_4" />
@@ -202,8 +201,9 @@
       </joint>
       <joint name="${prefix}joint_5" type="fixed">
-         <origin xyz="${M_SCALE*0} ${M_SCALE*-7} ${M_SCALE*0}" rpy="${M_PI/2} ${-M_PI/2} ${M_PI*0}" />
+         <origin xyz="${M_SCALE*0} ${M_SCALE*7} ${M_SCALE*0}" rpy="${-M_PI/2} ${-M_PI/2} ${M_PI*0}" />
          <parent link="${prefix}link_4" />
          <child link="${prefix}link_5" />
          <axis xyz="0 1 0" />
+         <limit lower="-0.31" upper="0.1" effort="0" velocity="0.5" />
       </joint>
       <joint name="${prefix}joint_6" type="prismatic">

Commit message: PhantomX Arm and Turtlebot Configuration added

File: phantomx_arm_description/urdf/phantomx.urdf (robot description, URDF)
Before this commit: robot phantomx_arm, 9 links, 8 joints
Links:
- removed link base_link
- removed link world
- added link arm_base_link, mass 1; collision mesh filename=package://phantomx_arm_description/meshes/collision/base_li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 scale=0.01 0.01 0.01; visual mesh filename=package://phantomx_arm_description/meshes/visual/base_link.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 scale=0.01 0.01 0.01
- link link_1: geometry collision mesh filename=package://phantomx_arm_description/meshes/collision/shoulde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 scale=0.01 0.01 0.01; visual mesh filename=package://phantomx_arm_description/meshes/visual/shoulder_l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 scale=0.01 0.01 0.01
- link link_2: geometry collision mesh filename=package://phantomx_arm_description/meshes/collision/bicep_l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 scale=0.01 0.01 0.01; visual mesh filename=package://phantomx_arm_description/meshes/visual/bicep_link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 scale=0.01 0.01 0.01
- link link_3: geometry collision mesh filename=package://phantomx_arm_description/meshes/collision/bicep_l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 scale=0.01 0.01 0.01; visual mesh filename=package://phantomx_arm_description/meshes/visual/bicep_link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 scale=0.01 0.01 0.01
- link link_4: geometry collision mesh filename=package://phantomx_arm_description/meshes/collision/wrist_l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 scale=0.01 0.01 0.01; visual mesh filename=package://phantomx_arm_description/meshes/visual/wrist_link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 scale=0.01 0.01 0.01
- link link_5: geometry collision mesh filename=package://phantomx_arm_description/meshes/collision/guide_r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 scale=0.01 0.01 0.01; visual mesh filename=package://phantomx_arm_description/meshes/visual/guide_rail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 scale=0.01 0.01 0.01
- link link_6: geometry collision mesh filename=package://phantomx_arm_description/meshes/collision/gripper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 scale=0.01 0.01 0.01; visual mesh filename=package://phantomx_arm_description/meshes/visual/gripper_ha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 scale=0.01 0.01 0.01
- link link_7: geometry collision mesh filename=package://phantomx_arm_description/meshes/collision/gripper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 scale=0.01 0.01 0.01; visual mesh filename=package://phantomx_arm_description/meshes/visual/gripper_ha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 scale=0.01 0.01 0.01
Joints:
- removed joint fixed
- added joint arm_base_joint: type fixed, parent plate_top_link, child arm_base_link, origin xyz=0.145 0.002 0.002 rpy=0.0 0.0 -1.570795, axis 0 1 0
- joint joint_1: origin xyz=0.005 -0.13 0.35 rpy=1.570795 6.28318 3.14159 -> xyz=0.00125 -0.0325 0.0875 rpy=1.570795 6.28318 3.14159; parent base_link -> arm_base_link
- joint joint_2: origin xyz=0.0 0.166 0.0 rpy=0 0 0 -> xyz=0.0 0.0415 0.0 rpy=0 0.0 0
- joint joint_3: origin xyz=0.0 0.4268 0.0 rpy=0 0 0 -> xyz=0.0 0.1067 0.0 rpy=0 0 0
- joint joint_4: origin xyz=0.0 0.4268 0.0 rpy=6.28318 6.28318 0 -> xyz=0.0 0.1067 0.0 rpy=6.28318 6.28318 0
- joint joint_5: origin xyz=0.0 0.28 0.0 rpy=-1.570795 -1.570795 0.0 -> xyz=0.0 0.07 0.0 rpy=-1.570795 -1.570795 0.0
- joint joint_6: origin xyz=0.14 0.0 0.0 rpy=-4.712385 6.28318 1.570795 -> xyz=0.035 0.0 0.0 rpy=-4.712385 6.28318 1.570795
- joint joint_7: origin xyz=-0.14 0.0 0.0 rpy=-4.712385 6.28318 -1.570795 -> xyz=-0.035 0.0 0.0 rpy=-4.712385 6.28318 -1.570795

File: phantomx_arm_description/urdf/phantomx_macro.xacro (robot description, xacro)
@@ -2,14 +2,14 @@
 <robot xmlns:xacro="http://ros.org/wiki/xacro">
    <property name="M_PI" value="3.14159"/>
-   <property name="M_SCALE" value="0.04"/>
+   <property name="M_SCALE" value="0.01"/>
    <xacro:include filename="$(find phantomx_arm_description)/urdf/common_materials.xacro" />
-   <link name="world" />
-   <joint name="fixed" type="fixed">
-      <parent link="world" />
-      <child link="base_link" />
-   </joint>
+   <!--link name="plate_top_link"/-->
+   <!--joint name="fixed" type="fixed">
+      <parent link="plate_top_link" />
+      <child link="ph_base_link" />
+   </joint-->
    <xacro:macro name="phantomx_arm" params="prefix">
       <!-- links -->
-      <link name="${prefix}base_link">
+      <link name="${prefix}arm_base_link">
          <visual>
             <origin xyz="${M_SCALE*10} ${M_SCALE*10} ${M_SCALE*0}" rpy="${M_PI*0} ${M_PI*0} ${M_PI}" />
@@ -172,7 +172,13 @@
       </link>
       <!-- joints -->
+      <joint name="${prefix}arm_base_joint" type="fixed">
+         <origin xyz="${M_SCALE*14.5} ${M_SCALE*0.2} ${M_SCALE*0.2}" rpy="${M_PI*0} ${M_PI*0} ${-M_PI/2}" />
+         <parent link="plate_top_link" />
+         <child link="${prefix}arm_base_link"/>
+         <axis xyz="0 1 0" />
+      </joint>
       <joint name="${prefix}joint_1" type="revolute">
          <origin xyz="${M_SCALE*0.125} ${M_SCALE*-3.25} ${M_SCALE*8.75}" rpy="${M_PI/2} ${M_PI*2} ${M_PI}" />
-         <parent link="${prefix}base_link" />
+         <parent link="${prefix}arm_base_link" />
          <child link="${prefix}link_1" />
          <axis xyz="0 1 0" />
@@ -180,5 +186,5 @@
       </joint>
       <joint name="${prefix}joint_2" type="revolute">
-         <origin xyz="${M_SCALE*0} ${M_SCALE*4.15} ${M_SCALE*0}" rpy="0 0 0" />
+         <origin xyz="${M_SCALE*0} ${M_SCALE*4.15} ${M_SCALE*0}" rpy="0 ${M_PI*0} 0" />
          <parent link="${prefix}link_1" />
          <child link="${prefix}link_2" />

Commit message: Update

File: phantomx_arm_description/urdf/phantomx.urdf (robot description, URDF)
Before this commit: robot phantomx_arm, 8 links, 8 joints
Joints:
- joint joint_6: type prismatic -> fixed
- joint joint_7: type prismatic -> fixed

File: phantomx_arm_description/urdf/phantomx_macro.xacro (robot description, xacro)
@@ -213,5 +213,5 @@
          <limit lower="-0.31" upper="0.1" effort="0" velocity="0.5" />
       </joint>
-      <joint name="${prefix}joint_6" type="prismatic">
+      <joint name="${prefix}joint_6" type="fixed">
          <origin xyz="${M_SCALE*3.5} ${M_SCALE*0} ${M_SCALE*0}" rpy="${-M_PI*1.5} ${M_PI*2} ${M_PI/2}" />
          <parent link="${prefix}link_5" />
@@ -220,5 +220,5 @@
          <limit lower="-0.31" upper="0.1" effort="0" velocity="0.5" />
       </joint>
-      <joint name="${prefix}joint_7" type="prismatic">
+      <joint name="${prefix}joint_7" type="fixed">
          <origin xyz="${M_SCALE*-3.5} ${M_SCALE*0} ${M_SCALE*0}" rpy="${-M_PI*1.5} ${M_PI*2} ${-M_PI/2}" />
          <parent link="${prefix}link_5" />
