Commit message: complete update

File: phantomx_arm_description/urdf/phantomx_macro.xacro (robot description, xacro)
@@ -52,5 +52,5 @@
       </link>
       <link name="${prefix}link_2">
-         <visual>with
+         <visual>
             <origin xyz="0 0 0" rpy="0 0 0" />
             <geometry>

Commit message: Make control of physical phantomx arm work
The gripper still needs to be manually controlled, need to test the gripper service better.
Also updated the phantomx urdf to match my mounting

File: phantomx_arm_description/urdf/phantomx_macro.xacro (robot description, xacro)
@@ -173,5 +173,5 @@
       <!-- joints -->
       <joint name="${prefix}arm_base_joint" type="fixed">
-         <origin xyz="${M_SCALE*14.5} ${M_SCALE*0.2} ${M_SCALE*0.2}" rpy="${M_PI*0} ${M_PI*0} ${-M_PI/2}" />
+         <origin xyz="${M_SCALE*12.25} ${M_SCALE*0.2} ${M_SCALE*0.2}" rpy="${M_PI*0} ${M_PI*0} ${-M_PI/2}" />
          <parent link="plate_top_link" />
          <child link="${prefix}arm_base_link"/>
@@ -179,5 +179,5 @@
       </joint>
       <joint name="${prefix}joint_1" type="revolute">
-         <origin xyz="${M_SCALE*0.125} ${M_SCALE*-3.25} ${M_SCALE*8.75}" rpy="${M_PI/2} ${M_PI*2} ${M_PI}" />
+         <origin xyz="${M_SCALE*0.125} ${M_SCALE*-3.25} ${M_SCALE*8.75}" rpy="${M_PI/2} ${M_PI*2} ${-M_PI/2}" />
          <parent link="${prefix}arm_base_link" />
          <child link="${prefix}link_1" />

Commit message: Correct collision surfaces to prevent the arm crashing into the base

File: phantomx_arm_description/urdf/phantomx_macro.xacro (robot description, xacro)
@@ -20,5 +20,5 @@
          </visual>
          <collision>
-            <origin xyz="0 0 0" rpy="0 0 0" />
+            <origin xyz="${M_SCALE*10} ${M_SCALE*10} ${M_SCALE*0}" rpy="${M_PI*0} ${M_PI*0} ${M_PI}" />
             <geometry>
                <mesh filename="package://phantomx_arm_description/meshes/collision/base_link.stl" scale="${M_SCALE} ${M_SCALE} ${M_SCALE}"/>
@@ -100,5 +100,5 @@
          </visual>
          <collision>
-            <origin xyz="0 0 0" rpy="0 0 0" />
+            <origin xyz="${M_SCALE*-1.18} ${M_SCALE*3.3} ${M_SCALE*0}" rpy="${M_PI*0} ${M_PI} ${-M_PI}" />
             <geometry>
                <mesh filename="package://phantomx_arm_description/meshes/collision/wrist_link.stl" scale="${M_SCALE} ${M_SCALE} ${M_SCALE}"/>
@@ -120,5 +120,5 @@
          </visual>
          <collision>
-            <origin xyz="0 0 0" rpy="0 0 0" />
+            <origin xyz="${M_SCALE*-1.15} ${M_SCALE*1.3} ${M_SCALE*-0.5}" rpy="0 0 0" />
             <geometry>
                <mesh filename="package://phantomx_arm_description/meshes/collision/guide_rail_fixed_link.stl" scale="${M_SCALE} ${M_SCALE} ${M_SCALE}"/>
@@ -140,5 +140,5 @@
          </visual>
          <collision>
-            <origin xyz="0 0 0" rpy="0 0 0" />
+            <origin xyz="${M_SCALE*-1.5} ${M_SCALE*-0.5} ${M_SCALE*0.5}" rpy="0 0 0" />
             <geometry>
                <mesh filename="package://phantomx_arm_description/meshes/collision/gripper_hand_fixed_link.stl" scale="${M_SCALE} ${M_SCALE} ${M_SCALE}"/>
@@ -160,5 +160,5 @@
          </visual>
          <collision>
-            <origin xyz="0 0 0" rpy="0 0 0" />
+            <origin xyz="${M_SCALE*-1.5} ${M_SCALE*-0.5} ${M_SCALE*0.5}" rpy="0 0 0" />
             <geometry>
                <mesh filename="package://phantomx_arm_description/meshes/collision/gripper_hand_fixed_link.stl" scale="${M_SCALE} ${M_SCALE} ${M_SCALE}"/>

Commit message: PhantomX Arm project Commit

File: phantomx_arm_description/urdf/phantomx_macro.xacro (robot description, xacro)
@@ -10,4 +10,15 @@
    </joint-->
    <xacro:macro name="phantomx_arm" params="prefix">
+      <!--
+	A Gazebo plugin needs to be added to your URDF that actually parses the transmission tags and loads the appropriate hardware interfaces and controller manager.
+        These plugins must inherit gazebo_ros_control::RobotHWSim which implements a simulated ros_control hardware_interface::RobotHW.
+	RobotHWSim provides API-level access to read and command joint properties in the Gazebo simulator.
+      -->
+      <gazebo>
+     	 <plugin name="gazebo_ros_control" filename="libgazebo_ros_control.so">
+           <robotNamespace>/phantomx_arm</robotNamespace>
+     	   <robotSimType>gazebo_ros_control/DefaultRobotHWSim</robotSimType>
+     	 </plugin>
+      </gazebo>
       <!-- links -->
       <link name="${prefix}arm_base_link">
@@ -155,5 +166,6 @@
             <origin xyz="${M_SCALE*-1.5} ${M_SCALE*-0.5} ${M_SCALE*0.5}" rpy="0 0 0" />
             <geometry>
-               <mesh filename="package://phantomx_arm_description/meshes/visual/gripper_hand_fixed_link.stl" scale="${M_SCALE} ${M_SCALE} ${M_SCALE}"/>
+            	<mesh filename="package://phantomx_arm_description/meshes/visual/gripper_hand_fixed_link.stl" scale="${M_SCALE} ${M_SCALE} ${M_SCALE}"/>
+<!-- box size="0.1 0.1 0.1"/ -->
             </geometry>
             <xacro:material_black />
@@ -162,5 +174,6 @@
             <origin xyz="${M_SCALE*-1.5} ${M_SCALE*-0.5} ${M_SCALE*0.5}" rpy="0 0 0" />
             <geometry>
-               <mesh filename="package://phantomx_arm_description/meshes/collision/gripper_hand_fixed_link.stl" scale="${M_SCALE} ${M_SCALE} ${M_SCALE}"/>
+<!-- box size="0.1 0.1 0.1"/ -->
+		<mesh filename="package://phantomx_arm_description/meshes/collision/gripper_hand_fixed_link.stl" scale="${M_SCALE} ${M_SCALE} ${M_SCALE}"/>
             </geometry>
          </collision>
@@ -183,5 +196,5 @@
          <child link="${prefix}link_1" />
          <axis xyz="0 1 0" />
-         <limit lower="-2.617" upper="2.617" effort="0" velocity="0.785" />
+         <limit lower="-2.617" upper="2.617" effort="17" velocity="0.785" />
       </joint>
       <joint name="${prefix}joint_2" type="revolute">
@@ -190,5 +203,5 @@
          <child link="${prefix}link_2" />
          <axis xyz="0 0 1" />
-         <limit lower="-2.617" upper="2.617" effort="0" velocity="1.571" />
+         <limit lower="-2.617" upper="2.617" effort="17" velocity="1.571" />
       </joint>
       <joint name="${prefix}joint_3" type="revolute">
@@ -197,5 +210,5 @@
          <child link="${prefix}link_3" />
          <axis xyz="0 0 1" />
-         <limit lower="-2.617" upper="2.617" effort="0" velocity="1.571" />
+         <limit lower="-2.617" upper="2.617" effort="17" velocity="1.571" />
       </joint>
       <joint name="${prefix}joint_4" type="revolute">
@@ -204,5 +217,5 @@
          <child link="${prefix}link_4" />
          <axis xyz="0 0 1" />
-         <limit lower="-1.745" upper="1.745" effort="0" velocity="1.571" />
+         <limit lower="-1.745" upper="1.745" effort="17" velocity="1.571" />
       </joint>
       <joint name="${prefix}joint_5" type="fixed">
@@ -211,5 +224,5 @@
          <child link="${prefix}link_5" />
          <axis xyz="0 1 0" />
-         <limit lower="-0.31" upper="0.1" effort="0" velocity="0.5" />
+         <limit lower="-0.31" upper="0.1" effort="17" velocity="0.5" />
       </joint>
       <joint name="${prefix}joint_6" type="fixed">
@@ -218,5 +231,5 @@
          <child link="${prefix}link_6" />
          <axis xyz="0 0 1" />
-         <limit lower="-0.31" upper="0.1" effort="0" velocity="0.5" />
+         <limit lower="-0.31" upper="0.1" effort="17" velocity="0.5" />
       </joint>
       <joint name="${prefix}joint_7" type="fixed">
@@ -225,10 +238,13 @@
          <child link="${prefix}link_7" />
          <axis xyz="0 0 1" />
-         <limit lower="-0.31" upper="0.1" effort="0" velocity="0.5" />
+         <limit lower="-0.31" upper="0.1" effort="17" velocity="0.5" />
       </joint>
    </xacro:macro>
+  <!-- hardware_interface::EffortJointInterface provides an appropriate hardware interface for our PhantomX Arm-->
   <transmission name="tran1">
     <type>transmission_interface/SimpleTransmission</type>
-    <joint name="joint_1"/>
+    <joint name="joint_1">
+	<hardwareInterface>EffortJointInterface</hardwareInterface>
+    </joint>
     <actuator name="motor1">
       <hardwareInterface>EffortJointInterface</hardwareInterface>
@@ -236,7 +252,10 @@
     </actuator>
   </transmission>
+ <!-- hardware_interface::EffortJointInterface provides an appropriate hardware interface for our PhantomX Arm-->
  <transmission name="tran2">
     <type>transmission_interface/SimpleTransmission</type>
-    <joint name="joint_2"/>
+    <joint name="joint_2">
+	<hardwareInterface>EffortJointInterface</hardwareInterface>
+    </joint>
     <actuator name="motor2">
       <hardwareInterface>EffortJointInterface</hardwareInterface>
@@ -244,7 +263,10 @@
     </actuator>
   </transmission>
+ <!-- hardware_interface::EffortJointInterface provides an appropriate hardware interface for our PhantomX Arm-->
  <transmission name="tran3">
     <type>transmission_interface/SimpleTransmission</type>
-    <joint name="joint_3"/>
+    <joint name="joint_3">
+	<hardwareInterface>EffortJointInterface</hardwareInterface>
+    </joint>
     <actuator name="motor3">
       <hardwareInterface>EffortJointInterface</hardwareInterface>
@@ -252,7 +274,10 @@
     </actuator>
   </transmission>
+ <!-- hardware_interface::EffortJointInterface provides an appropriate hardware interface for our PhantomX Arm-->
  <transmission name="tran4">
     <type>transmission_interface/SimpleTransmission</type>
-    <joint name="joint_4"/>
+    <joint name="joint_4">
+	<hardwareInterface>EffortJointInterface</hardwareInterface>
+    </joint>
     <actuator name="motor4">
       <hardwareInterface>EffortJointInterface</hardwareInterface>
@@ -260,7 +285,9 @@
     </actuator>
   </transmission>
- <transmission name="tran5">
-    <type>transmission_interface/SimpleTransmission</type>
-    <joint name="joint_6"/>
+ <!-- transmission name="tran5">
+    <type>transmission_interface/SimpleTransmission</type>
+    <joint name="joint_6">
+	<hardwareInterface>EffortJointInterface</hardwareInterface>
+    </joint>
     <actuator name="motor5">
       <hardwareInterface>EffortJointInterface</hardwareInterface>
@@ -270,9 +297,11 @@
  <transmission name="tran6">
     <type>transmission_interface/SimpleTransmission</type>
-    <joint name="joint_7"/>
+    <joint name="joint_7">
+	<hardwareInterface>EffortJointInterface</hardwareInterface>
+    </joint>
     <actuator name="motor6">
       <hardwareInterface>EffortJointInterface</hardwareInterface>
       <mechanicalReduction>1</mechanicalReduction>
     </actuator>
-  </transmission>
+  </transmission -->
 </robot>

File: phantomx_arm_turtlebot_description/urdf/stacks/hexagons.urdf.xacro (robot description, xacro)
@@ -207,4 +207,5 @@
         <geometry>
           <mesh filename="package://phantomx_arm_turtlebot_description/meshes/stacks/hexagons/plate_top.dae"/>
+<!-- box size="0.5 0.5 0.01"/ -->
         </geometry>
       </visual>
@@ -213,8 +214,9 @@
         <geometry>
 	 <mesh filename="package://phantomx_arm_turtlebot_description/meshes/stacks/hexagons/plate_top.dae"/>
-        </geometry>
-      </collision>
-      <inertial>
-        <mass value="0.01"/>
+<!-- box size="0.5 0.5 0.01"/ -->
+        </geometry>
+      </collision>
+      <inertial>
+        <mass value="1.0"/>
         <origin xyz="0 0 0"/>
         <inertia ixx="0.01" ixy="0.0" ixz="0.0"

Commit message: Added Maps for Boyd Sciences building in Gazebo

File: phantomx_arm_description/urdf/phantomx_macro.xacro (robot description, xacro)
@@ -9,4 +9,5 @@
       <child link="ph_base_link" />
    </joint-->
+   <!-- REFERENCE: http://answers.gazebosim.org/question/4372/the-inertia-matrix-explained/ -->
    <xacro:macro name="phantomx_arm" params="prefix">
       <!--
@@ -38,6 +39,6 @@
          <inertial>
             <origin xyz="0 0 0" rpy="0 0 0" />
-            <mass value="1" />
-            <inertia ixx="1.0" ixy="0.0" ixz="0.0" iyy="1.0" iyz="0.0" izz="1.0" />
+	    <mass value="0.005" />
+            <inertia ixx="0.005" ixy="0.0" ixz="0.0" iyy="0.005" iyz="0.0" izz="0.005" />
          </inertial>
       </link>
@@ -58,6 +59,6 @@
          <inertial>
             <origin xyz="0 0 0" rpy="0 0 0" />
-            <mass value="1" />
-            <inertia ixx="1.0" ixy="0.0" ixz="0.0" iyy="1.0" iyz="0.0" izz="1.0" />
+            <mass value="0.005" />
+            <inertia ixx="0.005" ixy="0.0" ixz="0.0" iyy="0.005" iyz="0.0" izz="0.005" />
          </inertial>
       </link>
@@ -78,6 +79,6 @@
          <inertial>
             <origin xyz="0 0 0" rpy="0 0 0" />
-            <mass value="1" />
-            <inertia ixx="1.0" ixy="0.0" ixz="0.0" iyy="1.0" iyz="0.0" izz="1.0" />
+            <mass value="0.005" />
+            <inertia ixx="0.005" ixy="0.0" ixz="0.0" iyy="0.005" iyz="0.0" izz="0.005" />
          </inertial>
       </link>
@@ -98,6 +99,6 @@
          <inertial>
             <origin xyz="0 0 0" rpy="0 0 0" />
-            <mass value="1" />
-            <inertia ixx="1.0" ixy="0.0" ixz="0.0" iyy="1.0" iyz="0.0" izz="1.0"/>
+            <mass value="0.005" />
+            <inertia ixx="0.005" ixy="0.0" ixz="0.0" iyy="0.005" iyz="0.0" izz="0.005"/>
          </inertial>
       </link>
@@ -118,6 +119,6 @@
          <inertial>
             <origin xyz="0 0 0" rpy="0 0 0" />
-            <mass value="1" />
-            <inertia ixx="1.0" ixy="0.0" ixz="0.0" iyy="1.0" iyz="0.0" izz="1.0" />
+            <mass value="0.005" />
+            <inertia ixx="0.005" ixy="0.0" ixz="0.0" iyy="0.005" iyz="0.0" izz="0.005" />
          </inertial>
       </link>
@@ -138,6 +139,6 @@
          <inertial>
             <origin xyz="0 0 0" rpy="0 0 0" />
-            <mass value="1" />
-            <inertia ixx="1.0" ixy="0.0" ixz="0.0" iyy="1.0" iyz="0.0" izz="1.0" />
+            <mass value="0.005" />
+            <inertia ixx="0.005" ixy="0.0" ixz="0.0" iyy="0.005" iyz="0.0" izz="0.005" />
          </inertial>
       </link>
@@ -158,6 +159,6 @@
          <inertial>
             <origin xyz="0 0 0" rpy="0 0 0" />
-            <mass value="1" />
-            <inertia ixx="1.0" ixy="0.0" ixz="0.0" iyy="1.0" iyz="0.0" izz="1.0" />
+            <mass value="0.005" />
+            <inertia ixx="0.005" ixy="0.0" ixz="0.0" iyy="0.005" iyz="0.0" izz="0.005" />
          </inertial>
       </link>
@@ -180,6 +181,6 @@
          <inertial>
             <origin xyz="0 0 0" rpy="0 0 0" />
-            <mass value="1" />
-            <inertia ixx="1.0" ixy="0.0" ixz="0.0" iyy="1.0" iyz="0.0" izz="1.0" />
+            <mass value="0.005" />
+            <inertia ixx="0.005" ixy="0.0" ixz="0.0" iyy="0.005" iyz="0.0" izz="0.005" />
          </inertial>
       </link>
@@ -196,5 +197,5 @@
          <child link="${prefix}link_1" />
          <axis xyz="0 1 0" />
-         <limit lower="-2.617" upper="2.617" effort="17" velocity="0.785" />
+         <limit lower="-2.617" upper="2.617" effort="3" velocity="0.785" />
       </joint>
       <joint name="${prefix}joint_2" type="revolute">
@@ -203,5 +204,5 @@
          <child link="${prefix}link_2" />
          <axis xyz="0 0 1" />
-         <limit lower="-2.617" upper="2.617" effort="17" velocity="1.571" />
+         <limit lower="-2.617" upper="2.617" effort="3" velocity="1.571" />
       </joint>
       <joint name="${prefix}joint_3" type="revolute">
@@ -210,5 +211,5 @@
          <child link="${prefix}link_3" />
          <axis xyz="0 0 1" />
-         <limit lower="-2.617" upper="2.617" effort="17" velocity="1.571" />
+         <limit lower="-2.617" upper="2.617" effort="3" velocity="1.571" />
       </joint>
       <joint name="${prefix}joint_4" type="revolute">
@@ -217,5 +218,5 @@
          <child link="${prefix}link_4" />
          <axis xyz="0 0 1" />
-         <limit lower="-1.745" upper="1.745" effort="17" velocity="1.571" />
+         <limit lower="-1.745" upper="1.745" effort="13" velocity="1.571" />
       </joint>
       <joint name="${prefix}joint_5" type="fixed">
@@ -224,5 +225,5 @@
          <child link="${prefix}link_5" />
          <axis xyz="0 1 0" />
-         <limit lower="-0.31" upper="0.1" effort="17" velocity="0.5" />
+         <limit lower="-0.31" upper="0.1" effort="13" velocity="0.5" />
       </joint>
       <joint name="${prefix}joint_6" type="fixed">
@@ -231,5 +232,5 @@
          <child link="${prefix}link_6" />
          <axis xyz="0 0 1" />
-         <limit lower="-0.31" upper="0.1" effort="17" velocity="0.5" />
+         <limit lower="-0.31" upper="0.1" effort="13" velocity="0.5" />
       </joint>
       <joint name="${prefix}joint_7" type="fixed">
@@ -238,5 +239,5 @@
          <child link="${prefix}link_7" />
          <axis xyz="0 0 1" />
-         <limit lower="-0.31" upper="0.1" effort="17" velocity="0.5" />
+         <limit lower="-0.31" upper="0.1" effort="13" velocity="0.5" />
       </joint>
    </xacro:macro>
