Commit message: Modified the URDF files to include multiple robot namespaces in Gazebo. The 'prefix' tags are used to pass the robot_namespace arguments down the chain of xacro files.

File: phantomx_arm_description/urdf/phantomx_macro.xacro (robot description, xacro)
@@ -4,4 +4,5 @@
    <property name="M_SCALE" value="0.01"/>
    <xacro:include filename="$(find phantomx_arm_description)/urdf/common_materials.xacro" />
+   <xacro:include filename="$(find phantomx_arm_description)/urdf/robot_name_description.xacro" />
    <!--link name="plate_top_link"/-->
    <!--joint name="fixed" type="fixed">
@@ -12,5 +13,6 @@
    <xacro:macro name="phantomx_arm" params="prefix">
       <!--
-	A Gazebo plugin needs to be added to your URDF that actually parses the transmission tags and loads the appropriate hardware interfaces and controller manager.
+	A Gazebo plugin needs to be added to your URDF that actually parses the transmission tags and loads the appropriate
+	hardware interfaces and controller manager.
         These plugins must inherit gazebo_ros_control::RobotHWSim which implements a simulated ros_control hardware_interface::RobotHW.
 	RobotHWSim provides API-level access to read and command joint properties in the Gazebo simulator.
@@ -18,10 +20,10 @@
       <gazebo>
      	 <plugin name="gazebo_ros_control" filename="libgazebo_ros_control.so">
-           <robotNamespace>/phantomx_arm</robotNamespace>
+           <robotNamespace>/${prefix}/phantomx_arm</robotNamespace>
      	   <robotSimType>gazebo_ros_control/DefaultRobotHWSim</robotSimType>
      	 </plugin>
       </gazebo>
       <!-- links -->
-      <link name="${prefix}arm_base_link">
+      <link name="arm_base_link">
          <visual>
             <origin xyz="${M_SCALE*10} ${M_SCALE*10} ${M_SCALE*0}" rpy="${M_PI*0} ${M_PI*0} ${M_PI}" />
@@ -43,5 +45,5 @@
          </inertial>
       </link>
-      <link name="${prefix}link_1">
+      <link name="link_1">
          <visual>
             <origin xyz="0 0 0" rpy="0 0 0" />
@@ -63,5 +65,5 @@
          </inertial>
       </link>
-      <link name="${prefix}link_2">
+      <link name="link_2">
          <visual>
             <origin xyz="0 0 0" rpy="0 0 0" />
@@ -83,5 +85,5 @@
          </inertial>
       </link>
-      <link name="${prefix}link_3">
+      <link name="link_3">
          <visual>
             <origin xyz="0 0 0" rpy="0 0 0" />
@@ -103,5 +105,5 @@
          </inertial>
       </link>
-      <link name="${prefix}link_4">
+      <link name="link_4">
          <visual>
             <origin xyz="${M_SCALE*-1.18} ${M_SCALE*3.3} ${M_SCALE*0}" rpy="${M_PI*0} ${M_PI} ${-M_PI}" />
@@ -123,5 +125,5 @@
          </inertial>
       </link>
-      <link name="${prefix}link_5">
+      <link name="link_5">
          <visual>
             <origin xyz="${M_SCALE*-1.15} ${M_SCALE*1.3} ${M_SCALE*-0.5}" rpy="0 0 0" />
@@ -143,5 +145,5 @@
          </inertial>
       </link>
-      <link name="${prefix}link_6">
+      <link name="link_6">
          <visual>
             <origin xyz="${M_SCALE*-1.5} ${M_SCALE*-0.5} ${M_SCALE*0.5}" rpy="0 0 0" />
@@ -163,5 +165,5 @@
          </inertial>
       </link>
-       <link name="${prefix}link_7">
+       <link name="link_7">
          <visual>
             <origin xyz="${M_SCALE*-1.5} ${M_SCALE*-0.5} ${M_SCALE*0.5}" rpy="0 0 0" />
@@ -186,56 +188,56 @@
       </link>
       <!-- joints -->
-      <joint name="${prefix}arm_base_joint" type="fixed">
+      <joint name="arm_base_joint" type="fixed">
          <origin xyz="${M_SCALE*12.25} ${M_SCALE*0.2} ${M_SCALE*0.2}" rpy="${M_PI*0} ${M_PI*0} ${-M_PI/2}" />
          <parent link="plate_top_link" />
-         <child link="${prefix}arm_base_link"/>
+         <child link="arm_base_link"/>
          <axis xyz="0 1 0" />
       </joint>
-      <joint name="${prefix}joint_1" type="revolute">
+      <joint name="joint_1" type="revolute">
          <origin xyz="${M_SCALE*0.125} ${M_SCALE*-3.25} ${M_SCALE*8.75}" rpy="${M_PI/2} ${M_PI*2} ${-M_PI/2}" />
-         <parent link="${prefix}arm_base_link" />
-         <child link="${prefix}link_1" />
+         <parent link="arm_base_link" />
+         <child link="link_1" />
          <axis xyz="0 1 0" />
          <limit lower="-2.617" upper="2.617" effort="3" velocity="0.785" />
       </joint>
-      <joint name="${prefix}joint_2" type="revolute">
+      <joint name="joint_2" type="revolute">
          <origin xyz="${M_SCALE*0} ${M_SCALE*4.15} ${M_SCALE*0}" rpy="0 ${M_PI*0} 0" />
-         <parent link="${prefix}link_1" />
-         <child link="${prefix}link_2" />
+         <parent link="link_1" />
+         <child link="link_2" />
          <axis xyz="0 0 1" />
          <limit lower="-2.617" upper="2.617" effort="3" velocity="1.571" />
       </joint>
-      <joint name="${prefix}joint_3" type="revolute">
+      <joint name="joint_3" type="revolute">
          <origin xyz="${M_SCALE*0} ${M_SCALE*10.67} ${M_SCALE*0}" rpy="0 0 0" />
-         <parent link="${prefix}link_2" />
-         <child link="${prefix}link_3" />
+         <parent link="link_2" />
+         <child link="link_3" />
          <axis xyz="0 0 1" />
          <limit lower="-2.617" upper="2.617" effort="3" velocity="1.571" />
       </joint>
-      <joint name="${prefix}joint_4" type="revolute">
+      <joint name="joint_4" type="revolute">
          <origin xyz="${M_SCALE*0} ${M_SCALE*10.67} ${M_SCALE*0}" rpy="${M_PI*2} ${M_PI*2} 0" />
-         <parent link="${prefix}link_3" />
-         <child link="${prefix}link_4" />
+         <parent link="link_3" />
+         <child link="link_4" />
          <axis xyz="0 0 1" />
          <limit lower="-1.745" upper="1.745" effort="13" velocity="1.571" />
       </joint>
-      <joint name="${prefix}joint_5" type="fixed">
+      <joint name="joint_5" type="fixed">
          <origin xyz="${M_SCALE*0} ${M_SCALE*7} ${M_SCALE*0}" rpy="${-M_PI/2} ${-M_PI/2} ${M_PI*0}" />
-         <parent link="${prefix}link_4" />
-         <child link="${prefix}link_5" />
+         <parent link="link_4" />
+         <child link="link_5" />
          <axis xyz="0 1 0" />
          <limit lower="-0.31" upper="0.1" effort="13" velocity="0.5" />
       </joint>
-      <joint name="${prefix}joint_6" type="fixed">
+      <joint name="joint_6" type="fixed">
          <origin xyz="${M_SCALE*3.5} ${M_SCALE*0} ${M_SCALE*0}" rpy="${-M_PI*1.5} ${M_PI*2} ${M_PI/2}" />
-         <parent link="${prefix}link_5" />
-         <child link="${prefix}link_6" />
+         <parent link="link_5" />
+         <child link="link_6" />
          <axis xyz="0 0 1" />
          <limit lower="-0.31" upper="0.1" effort="13" velocity="0.5" />
       </joint>
-      <joint name="${prefix}joint_7" type="fixed">
+      <joint name="joint_7" type="fixed">
          <origin xyz="${M_SCALE*-3.5} ${M_SCALE*0} ${M_SCALE*0}" rpy="${-M_PI*1.5} ${M_PI*2} ${-M_PI/2}" />
-         <parent link="${prefix}link_5" />
-         <child link="${prefix}link_7" />
+         <parent link="link_5" />
+         <child link="link_7" />
          <axis xyz="0 0 1" />
          <limit lower="-0.31" upper="0.1" effort="13" velocity="0.5" />

File: phantomx_arm_turtlebot_description/robots/kobuki_hexagons_kinect.urdf.xacro (robot description, xacro)
@@ -6,5 +6,11 @@
 -->
 <robot name="turtlebot" xmlns:xacro="http://ros.org/wiki/xacro">
-  <xacro:include filename="$(find phantomx_arm_turtlebot_description)/urdf/turtlebot_library.urdf.xacro" />
+  <!-- Turtlebot Kobuki Description Files -->
+  <xacro:include filename="$(find phantomx_arm_turtlebot_description)/urdf/turtlebot_library.urdf.xacro"/>
+  <!-- PhantomX Arm -->
+  <!-- For convenience and effective use of multiple namespaces, this call has been moved to kobuki_hexagons_kinect.urdf.xacro -->
+  <!-- The 'prefix' tag for the 'phantomx_arm' macro allows robot_ns reference to be sent to the urdf.xacro files directly from our launch files -->
+  <xacro:include filename="$(find phantomx_arm_description)/urdf/phantomx_macro.xacro"/>
+  <xacro:phantomx_arm prefix="$(arg prefix)"/>
   <kobuki/>
   <stack_hexagons parent="base_link"/>

File: phantomx_arm_turtlebot_description/urdf/turtlebot_library.urdf.xacro (robot description, xacro)
@@ -17,4 +17,5 @@
   <xacro:include filename="$(find phantomx_arm_turtlebot_description)/urdf/sensors/asus_xtion_pro.urdf.xacro"/>
   <!-- PhantomX Arm -->
- <xacro:include filename="$(find phantomx_arm_description)/urdf/phantomx.xacro"/>
+  <!-- For convenience and effective use of multiple namespaces, this call has been moved to kobuki_hexagons_kinect.urdf.xacro -->
+  <!-- xacro:include filename="$(find phantomx_arm_description)/urdf/${prefix}.xacro"/ -->
 </robot>

Commit message: Improved precision for the multiple phantomx turtlebot arm_controllers in Gazebo

File: phantomx_arm_description/urdf/phantomx_macro.xacro (robot description, xacro)
@@ -229,17 +229,17 @@
          <limit lower="-0.31" upper="0.1" effort="13" velocity="0.5" />
       </joint>
-      <joint name="joint_6" type="fixed">
+      <joint name="joint_6" type="prismatic">
          <origin xyz="${M_SCALE*3.5} ${M_SCALE*0} ${M_SCALE*0}" rpy="${-M_PI*1.5} ${M_PI*2} ${M_PI/2}" />
          <parent link="link_5" />
          <child link="link_6" />
          <axis xyz="0 0 1" />
-         <limit lower="-0.31" upper="0.1" effort="13" velocity="0.5" />
-      </joint>
-      <joint name="joint_7" type="fixed">
+         <limit lower="-0.02" upper="0.0" effort="13" velocity="0.5" />
+      </joint>
+      <joint name="joint_7" type="prismatic">
          <origin xyz="${M_SCALE*-3.5} ${M_SCALE*0} ${M_SCALE*0}" rpy="${-M_PI*1.5} ${M_PI*2} ${-M_PI/2}" />
          <parent link="link_5" />
          <child link="link_7" />
          <axis xyz="0 0 1" />
-         <limit lower="-0.31" upper="0.1" effort="13" velocity="0.5" />
+         <limit lower="-0.02" upper="0.0" effort="13" velocity="0.5" />
       </joint>
    </xacro:macro>
@@ -288,5 +288,6 @@
     </actuator>
   </transmission>
- <!-- transmission name="tran5">
+ <!-- hardware_interface::EffortJointInterface provides an appropriate hardware interface for our PhantomX Arm-->
+ <transmission name="tran5">
     <type>transmission_interface/SimpleTransmission</type>
     <joint name="joint_6">
@@ -298,4 +299,5 @@
     </actuator>
   </transmission>
+ <!-- hardware_interface::EffortJointInterface provides an appropriate hardware interface for our PhantomX Arm-->
  <transmission name="tran6">
     <type>transmission_interface/SimpleTransmission</type>
@@ -307,4 +309,4 @@
       <mechanicalReduction>1</mechanicalReduction>
     </actuator>
-  </transmission -->
+  </transmission>
 </robot>

Commit message: Modifying the PhantomX Macro files for some tests

File: phantomx_arm_description/urdf/phantomx_macro.xacro (robot description, xacro)
@@ -20,8 +20,12 @@
       <gazebo>
      	 <plugin name="gazebo_ros_control" filename="libgazebo_ros_control.so">
-           <robotNamespace>/${prefix}/phantomx_arm</robotNamespace>
+           <!-- robotNamespace>/${prefix}/phantomx_arm</robotNamespace-->
 	   <robotSimType>gazebo_ros_control/DefaultRobotHWSim</robotSimType>
      	 </plugin>
       </gazebo>
+      <!--gazebo reference="link_7">
+     	 <plugin name="model_push" filename="libmodel_push.so">
+     	 </plugin>
+      </gazebo-->
       <!-- links -->
       <link name="arm_base_link">
@@ -206,5 +210,5 @@
          <child link="link_2" />
          <axis xyz="0 0 1" />
-         <limit lower="-2.617" upper="2.617" effort="3" velocity="1.571" />
+         <limit lower="-2.617" upper="2.617" effort="3" velocity="1.071" />
       </joint>
       <joint name="joint_3" type="revolute">
@@ -213,5 +217,5 @@
          <child link="link_3" />
          <axis xyz="0 0 1" />
-         <limit lower="-2.617" upper="2.617" effort="3" velocity="1.571" />
+         <limit lower="-2.617" upper="2.617" effort="3" velocity="1.071" />
       </joint>
       <joint name="joint_4" type="revolute">
@@ -220,5 +224,5 @@
          <child link="link_4" />
          <axis xyz="0 0 1" />
-         <limit lower="-1.745" upper="1.745" effort="13" velocity="1.571" />
+         <limit lower="-1.745" upper="1.745" effort="13" velocity="1.071" />
       </joint>
       <joint name="joint_5" type="fixed">
@@ -227,5 +231,5 @@
          <child link="link_5" />
          <axis xyz="0 1 0" />
-         <limit lower="-0.31" upper="0.1" effort="13" velocity="0.5" />
+         <limit lower="-0.31" upper="0.1" effort="13" velocity="0.065" />
       </joint>
       <joint name="joint_6" type="prismatic">
@@ -234,5 +238,6 @@
          <child link="link_6" />
          <axis xyz="0 0 1" />
-         <limit lower="-0.02" upper="0.0" effort="13" velocity="0.5" />
+         <limit lower="-0.02" upper="0.0" effort="3" velocity="0.065" />
+	 <mimic joint="joint_7" multiplier="-1" offset="0"/>
       </joint>
       <joint name="joint_7" type="prismatic">
@@ -241,5 +246,5 @@
          <child link="link_7" />
          <axis xyz="0 0 1" />
-         <limit lower="-0.02" upper="0.0" effort="13" velocity="0.5" />
+         <limit lower="-0.02" upper="0.0" effort="3" velocity="0.065" />
       </joint>
    </xacro:macro>

Commit message: Modified the World environment in order to better exploit the strengths of our algorithm

File: phantomx_arm_description/urdf/phantomx_macro.xacro (robot description, xacro)
@@ -58,4 +58,44 @@
     	 </inertial>
       </link>
+      <link name="phantomx_Flag_link_1">
+         <visual>
+            <origin xyz="0.1 0.1 0.2050" rpy="${M_PI*0} ${M_PI*0} ${M_PI}" />
+            <geometry>
+              <box size = "0.01 0.01 0.395" />
+            </geometry>
+	    <xacro:material_black />
+         </visual>
+         <collision>
+            <origin xyz="0.1 0.1 0.2050" rpy="${M_PI*0} ${M_PI*0} ${M_PI}" />
+            <geometry>
+              <box size = "0.01 0.01 0.395" />
+            </geometry>
+         </collision>
+         <inertial>
+            <origin xyz="0 0 0" rpy="0 0 0" />
+	    <mass value="0.005" />
+            <inertia ixx="0.005" ixy="0.0" ixz="0.0" iyy="0.005" iyz="0.0" izz="0.005" />
+         </inertial>
+      </link>
+      <link name="phantomx_Flag_link_2">
+         <visual>
+            <origin xyz="0.09 0.1 0.35" rpy="${M_PI*0} ${M_PI*0} ${M_PI}" />
+            <geometry>
+              <box size = "0.15 0.01 0.1" />
+            </geometry>
+	    <xacro:material_black />
+         </visual>
+         <collision>
+            <origin xyz="0.09 0.1 0.35" rpy="${M_PI*0} ${M_PI*0} ${M_PI}" />
+            <geometry>
+              <box size = "0.15 0.01 0.1" />
+            </geometry>
+         </collision>
+         <inertial>
+            <origin xyz="0 0 0" rpy="0 0 0" />
+	    <mass value="0.005" />
+            <inertia ixx="0.005" ixy="0.0" ixz="0.0" iyy="0.005" iyz="0.0" izz="0.005" />
+         </inertial>
+      </link>
       <link name="arm_base_link">
          <visual>
@@ -226,4 +266,16 @@
     	 <parent link="plate_top_link"/>
          <child link="phantomx_camera_link"/>
+      </joint>
+      <joint name="phantomx_Flag_joint_1" type="fixed">
+    	 <axis xyz="0 1 0" />
+    	 <origin xyz="-0.2 -0.1 -0.0087" rpy="0 0 0"/>
+    	 <parent link="plate_top_link"/>
+         <child link="phantomx_Flag_link_1"/>
+      </joint>
+      <joint name="phantomx_Flag_joint_2" type="fixed">
+    	 <axis xyz="0 1 0" />
+    	 <origin xyz="-0.27 -0.1 -0.0087" rpy="0 0 0"/>
+    	 <parent link="plate_top_link"/>
+         <child link="phantomx_Flag_link_2"/>
       </joint>
       <joint name="arm_base_joint" type="fixed">
