Commit message: Make the collision surface more accurate for the turtlebot 2's hexagons

File: phantomx_arm_turtlebot_description/urdf/stacks/hexagons.urdf.xacro (robot description, xacro)
@@ -212,5 +212,5 @@
         <origin xyz="0.01364 0 0" rpy="0 0 0"/>
         <geometry>
-          <cylinder length="0.006" radius="0.170"/>
+	 <mesh filename="package://phantomx_arm_turtlebot_description/meshes/stacks/hexagons/plate_top.dae"/>
         </geometry>
       </collision>
